Commit message: added turtlebot with kinect

File: hector_quadrotor_description/urdf/kinect_camera.urdf.xacro (robot description, xacro)
@@ -14,5 +14,5 @@
           <inertia ixx="0.000000017" ixy="0" ixz="0" iyy="0.000000017" iyz="0" izz="0.000000017" />
         </inertial>
-        <!--<xacro:inertial_sphere mass="0.01" diameter="0.07" />
+        <!-- <xacro:inertial_sphere mass="0.01" diameter="0.07" /> -->
         <visual>
           <origin xyz="0 0 0" rpy="0 0 0" />
@@ -21,10 +21,10 @@
           </geometry>
         </visual>
-        <collision>
+         <collision>
           <origin xyz="0 0 0" rpy="0 0 0" />
           <geometry>
             <mesh filename="package://hector_sensors_description/meshes/kinect_camera/kinect_camera_simple.stl"/>
           </geometry>
-        </collision>-->
+        </collision>
       </link>
       <joint name="${name}_depth_joint" type="fixed">

Commit message: add turtle

File: hector_quadrotor_description/urdf/kinect_camera.urdf.xacro (robot description, xacro)
@@ -15,5 +15,5 @@
         </inertial>
         <!-- <xacro:inertial_sphere mass="0.01" diameter="0.07" /> -->
-        <visual>
+        <!-- <visual>
           <origin xyz="0 0 0" rpy="0 0 0" />
           <geometry>
@@ -26,5 +26,5 @@
             <mesh filename="package://hector_sensors_description/meshes/kinect_camera/kinect_camera_simple.stl"/>
           </geometry>
-        </collision>
+        </collision> -->
       </link>
       <joint name="${name}_depth_joint" type="fixed">

File: hector_quadrotor_description/urdf/turtlebot.urdf.xacro (robot description, xacro)
@@ -11,5 +11,5 @@
   <xacro:include filename="$(find hector_quadrotor_description)/urdf/kinect_camera.urdf.xacro" />
   <xacro:kinect_camera name="camera" parent="base_link">
-    <origin xyz="0.15 0.0 0.2" rpy="0 0 0"/>
+    <origin xyz="0.15 0.0 0.5" rpy="0 0 0"/>
   </xacro:kinect_camera>
   <kobuki/>

Commit message: update

File: hector_quadrotor_description/urdf/kinect_camera.urdf.xacro (robot description, xacro)
@@ -9,5 +9,5 @@
       </joint>
       <link name="${name}_link">
-	      <inertial>
+        <inertial>
           <mass value="0.01" />
           <origin xyz="0 0 0" rpy="0 0 0" />
@@ -73,5 +73,5 @@
             <clip>
               <near>0.01</near>
-	            <far>100</far> <!--changed from 100 to 1000-->
+              <far>100</far> <!--changed from 100 to 1000-->
             </clip>
           </camera>
@@ -86,6 +86,6 @@
           </plugin>
         </sensor>
-      	<turnGravityOff>true</turnGravityOff>
+        <turnGravityOff>true</turnGravityOff>
       </gazebo>
     </xacro:macro>
-  </robot>
+</robot>

File: hector_quadrotor_description/urdf/quadrotor_with_multiple_kinects.urdf.xacro (robot description, xacro)
@@ -17,18 +17,18 @@
     </xacro:kinect_camera>
     <include filename="$(find hector_quadrotor_description)/urdf/kinect_camera.urdf.xacro" />
-    <xacro:kinect_camera name="kinect_right_30" parent="base_link">
+    <xacro:kinect_camera name="kinect_right" parent="base_link">
       <origin xyz="0.1 0.0 0.1" rpy="0 0 ${-30*M_PI/180}"/>
     </xacro:kinect_camera>
-    <include filename="$(find hector_quadrotor_description)/urdf/kinect_camera.urdf.xacro" />
+    <!-- <include filename="$(find hector_quadrotor_description)/urdf/kinect_camera.urdf.xacro" />
     <xacro:kinect_camera name="kinect_right_60" parent="base_link">
       <origin xyz="0.1 0.0 0.1" rpy="0 0 ${-60*M_PI/180}"/>
-    </xacro:kinect_camera>
+    </xacro:kinect_camera>-->
     <include filename="$(find hector_quadrotor_description)/urdf/kinect_camera.urdf.xacro" />
-    <xacro:kinect_camera name="kinect_left_30" parent="base_link">
+    <xacro:kinect_camera name="kinect_left" parent="base_link">
       <origin xyz="0.1 0.0 0.1" rpy="0 0 ${30*M_PI/180}"/>
     </xacro:kinect_camera>
-    <include filename="$(find hector_quadrotor_description)/urdf/kinect_camera.urdf.xacro" />
+<!--     <include filename="$(find hector_quadrotor_description)/urdf/kinect_camera.urdf.xacro" />
     <xacro:kinect_camera name="kinect_left_60" parent="base_link">
       <origin xyz="0.1 0.0 0.1" rpy="0 0 ${60*M_PI/180}"/>
-    </xacro:kinect_camera>
+    </xacro:kinect_camera> -->
 </robot>
