Commit message: update: change quadcopter

File: hector_quadrotor_description/urdf/quadrotor.gazebo.xacro (robot description, xacro)
@@ -1,5 +1,6 @@
 <?xml version="1.0"?>
 <robot name="quadrotor" xmlns:xacro="http://www.ros.org/wiki/xacro">
-    <xacro:include filename="$(find hector_quadrotor_description)/urdf/quadrotor.urdf.xacro" />
+    <xacro:include filename="$(find hector_quadrotor_description)/urdf/quadrotor_with_cam_and_kinect.urdf.xacro" />
+    <!-- <xacro:include filename="$(find hector_quadrotor_description)/urdf/quadrotor.urdf.xacro" /> -->
     <xacro:include filename="$(find hector_quadrotor_gazebo)/urdf/quadrotor_plugins.gazebo.xacro" />
 </robot>

File: hector_quadrotor_description/urdf/quadrotor_with_cam_and_kinect.urdf.xacro (robot description, xacro)
@@ -1,9 +1,11 @@
 <?xml version="1.0"?>
-<robot name="quadrotor" xmlns:xacro="http://www.ros.org/wiki/xacro">
-    <xacro:property name="M_PI" value="3.1415926535897931" />
+<robot
+    name="quadrotor"
+    xmlns:xacro="http://www.ros.org/wiki/xacro"
+>
+    <!-- <xacro:property name="M_PI" value="3.1415926535897931" /> -->
     <!-- Included URDF Files -->
     <xacro:include filename="$(find hector_quadrotor_description)/urdf/ardrone_base.urdf.xacro" />
-    <!-- Instantiate quadrotor_base_macro once (has no parameters atm) -->
-    <xacro:quadrotor_base_macro />
+    <!-- <xacro:include filename="$(find hector_quadrotor_description)/urdf/quadrotor_base.urdf.xacro" /> -->
     <!-- Forward facing camera
     <xacro:include filename="$(find hector_sensors_description)/urdf/generic_camera.urdf.xacro" />
@@ -32,3 +34,5 @@
       <origin xyz="0.1 0.0 0.1" rpy="0 0 ${60*M_PI/180}"/>
     </xacro:kinect_camera>-->
+    <!-- Instantiate quadrotor_base_macro once (has no parameters atm) -->
+    <xacro:quadrotor_base_macro />
 </robot>
